Commit message: made atlas_minimal_contact less minimal

File: examples/Atlas/urdf/atlas_minimal_contact.urdf (robot description, URDF)
Before this commit: robot atlas, 45 links, 44 joints
Links:
- added link l_hand_camera_link
- added link l_hand_camera_optical_frame
- added link l_hand_face
- added link l_hand_force_torque, mass 0.1; visual box size=0.01 0.01 0.01
- added link l_hand_gripper
- added link left_finger_1_link_0; visual mesh filename=package://Atlas/urdf/meshes/s-model_articulated/visual/link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
- added link left_finger_1_link_1; visual mesh filename=package://Atlas/urdf/meshes/s-model_articulated/visual/link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
- added link left_finger_1_link_2; visual mesh filename=package://Atlas/urdf/meshes/s-model_articulated/visual/link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
- added link left_finger_1_link_3; visual mesh filename=package://Atlas/urdf/meshes/s-model_articulated/visual/link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
- added link left_finger_2_link_0; visual mesh filename=package://Atlas/urdf/meshes/s-model_articulated/visual/link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
- added link left_finger_2_link_1; visual mesh filename=package://Atlas/urdf/meshes/s-model_articulated/visual/link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
- added link left_finger_2_link_2; visual mesh filename=package://Atlas/urdf/meshes/s-model_articulated/visual/link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
- added link left_finger_2_link_3; visual mesh filename=package://Atlas/urdf/meshes/s-model_articulated/visual/link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
- added link left_finger_middle_link_0; visual mesh filename=package://Atlas/urdf/meshes/s-model_articulated/visual/link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
- added link left_finger_middle_link_1; visual mesh filename=package://Atlas/urdf/meshes/s-model_articulated/visual/link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
- added link left_finger_middle_link_2; visual mesh filename=package://Atlas/urdf/meshes/s-model_articulated/visual/link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
- added link left_finger_middle_link_3; visual mesh filename=package://Atlas/urdf/meshes/s-model_articulated/visual/link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
- added link left_palm; visual mesh filename=package://Atlas/urdf/meshes/s-model_articulated/visual/palm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
- added link r_hand_camera_link
- added link r_hand_camera_optical_frame
- added link r_hand_face
- added link r_hand_force_torque, mass 0.1; visual box size=0.01 0.01 0.01
- added link r_hand_gripper
- added link right_finger_1_link_0; visual mesh filename=package://Atlas/urdf/meshes/s-model_articulated/visual/link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
- added link right_finger_1_link_1; visual mesh filename=package://Atlas/urdf/meshes/s-model_articulated/visual/link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
- added link right_finger_1_link_2; visual mesh filename=package://Atlas/urdf/meshes/s-model_articulated/visual/link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
- added link right_finger_1_link_3; visual mesh filename=package://Atlas/urdf/meshes/s-model_articulated/visual/link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
- added link right_finger_2_link_0; visual mesh filename=package://Atlas/urdf/meshes/s-model_articulated/visual/link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
- added link right_finger_2_link_1; visual mesh filename=package://Atlas/urdf/meshes/s-model_articulated/visual/link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
- added link right_finger_2_link_2; visual mesh filename=package://Atlas/urdf/meshes/s-model_articulated/visual/link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
- added link right_finger_2_link_3; visual mesh filename=package://Atlas/urdf/meshes/s-model_articulated/visual/link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
- added link right_finger_middle_link_0; visual mesh filename=package://Atlas/urdf/meshes/s-model_articulated/visual/link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
- added link right_finger_middle_link_1; visual mesh filename=package://Atlas/urdf/meshes/s-model_articulated/visual/link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
- added link right_finger_middle_link_2; visual mesh filename=package://Atlas/urdf/meshes/s-model_articulated/visual/link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
- added link right_finger_middle_link_3; visual mesh filename=package://Atlas/urdf/meshes/s-model_articulated/visual/link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
- added link right_palm; visual mesh filename=package://Atlas/urdf/meshes/s-model_articulated/visual/palm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
- link l_hand: geometry collision sphere radius=0; collision sphere radius=0
- link l_lleg: geometry collision sphere radius=0; visual mesh filename=package://Atlas/urdf/meshes/l_lleg.obj
- link l_uleg: geometry collision sphere radius=0; collision sphere radius=0
- link pelvis: geometry collision sphere radius=0; collision sphere radius=0
- link r_hand: geometry collision sphere radius=0; collision sphere radius=0
- link r_lleg: geometry collision sphere radius=0; visual mesh filename=package://Atlas/urdf/meshes/r_lleg.obj
- link r_uleg: geometry collision sphere radius=0; collision sphere radius=0
- link utorso: geometry collision sphere radius=0; collision sphere radius=0
Joints:
- added joint l_hand_camera_joint: type fixed, parent l_hand_force_torque, child l_hand_camera_link, origin xyz=-0.09892  0.01431 0.0 rpy= -1.57079 0  1.5708
- added joint l_hand_camera_optical_frame_joint: type fixed, parent l_hand_camera_link, child l_hand_camera_optical_frame, origin xyz=0 0 0 rpy=-1.57079 0.0 -1.57079
- added joint l_hand_face_joint: type fixed, parent l_hand_force_torque, child l_hand_face, origin xyz=0 0.12 0 rpy=0.0 0.0 0.0
- added joint l_hand_force_torque_joint: type fixed, parent l_hand, child l_hand_force_torque, origin xyz=0 -0.1245 0 rpy=0 0 3.141592
- added joint l_hand_gripper_joint: type fixed, parent l_hand_force_torque, child l_hand_gripper, origin xyz=0 0.18 0 rpy=0.0 0.0 0.0
- added joint left_finger_1_joint_1: type fixed, parent left_finger_1_link_0, child left_finger_1_link_1, origin xyz=0.020 0 0 rpy=0 0 0, axis 0 0 1, limit lower=0 upper=3.1416 effort=100 velocity=100
- added joint left_finger_1_joint_2: type fixed, parent left_finger_1_link_1, child left_finger_1_link_2, origin xyz=0.050 -.028 0 rpy=0 0 -0.52, axis 0 0 1, limit lower=0 upper=3.1416 effort=100 velocity=100
- added joint left_finger_1_joint_3: type fixed, parent left_finger_1_link_2, child left_finger_1_link_3, origin xyz=0.039 0 0 rpy=0 0 0, axis 0 0 1, limit lower=0 upper=3.1416 effort=100 velocity=100
- added joint left_finger_2_joint_1: type fixed, parent left_finger_2_link_0, child left_finger_2_link_1, origin xyz=0.020 0 0 rpy=0 0 0, axis 0 0 1, limit lower=0 upper=3.1416 effort=100 velocity=100
- added joint left_finger_2_joint_2: type fixed, parent left_finger_2_link_1, child left_finger_2_link_2, origin xyz=0.050 -.028 0 rpy=0 0 -0.52, axis 0 0 1, limit lower=0 upper=3.1416 effort=100 velocity=100
- added joint left_finger_2_joint_3: type fixed, parent left_finger_2_link_2, child left_finger_2_link_3, origin xyz=0.039 0 0 rpy=0 0 0, axis 0 0 1, limit lower=0 upper=3.1416 effort=100 velocity=100
- added joint left_finger_middle_joint_1: type fixed, parent left_finger_middle_link_0, child left_finger_middle_link_1, origin xyz=0.020 0 0 rpy=0 0 0, axis 0 0 1, limit lower=0 upper=3.1416 effort=100 velocity=100
- added joint left_finger_middle_joint_2: type fixed, parent left_finger_middle_link_1, child left_finger_middle_link_2, origin xyz=0.050 -.028 0 rpy=0 0 -0.52, axis 0 0 1, limit lower=0 upper=3.1416 effort=100 velocity=100
- added joint left_finger_middle_joint_3: type fixed, parent left_finger_middle_link_2, child left_finger_middle_link_3, origin xyz=0.039 0 0 rpy=0 0 0, axis 0 0 1, limit lower=0 upper=3.1416 effort=100 velocity=100
- added joint left_palm_finger_1_joint: type fixed, parent left_palm, child left_finger_1_link_0, origin xyz=-0.0455 0.0214 0.036 rpy=0 3.1416 -1.57, axis 0 1 0, limit lower=-0.16 upper=0.25 effort=100 velocity=100
- added joint left_palm_finger_2_joint: type fixed, parent left_palm, child left_finger_2_link_0, origin xyz=-0.0455 0.0214 -0.036 rpy=0 3.1416 -1.57, axis 0 1 0, limit lower=-0.25 upper=0.16 effort=100 velocity=100
- added joint left_palm_finger_middle_joint: type fixed, parent left_palm, child left_finger_middle_link_0, origin xyz=0.0455 0.0214 0 rpy=0 0 1.57, axis 0 0 1
- added joint left_robotiq_hand_joint: type fixed, parent l_hand_force_torque, child left_palm, origin xyz=0 0.06566 0.0 rpy=0 -1.57079 0
- added joint r_hand_camera_joint: type fixed, parent r_hand_force_torque, child r_hand_camera_link, origin xyz=0.09892  0.01431 0.0 rpy= 1.57079 0  1.5708
- added joint r_hand_camera_optical_frame_joint: type fixed, parent r_hand_camera_link, child r_hand_camera_optical_frame, origin xyz=0 0 0 rpy=-1.57079 0.0 -1.57079
- added joint r_hand_face_joint: type fixed, parent r_hand_force_torque, child r_hand_face, origin xyz=0 0.12 0 rpy=0.0 0.0 0.0
- added joint r_hand_force_torque_joint: type fixed, parent r_hand, child r_hand_force_torque, origin xyz=0 -0.1245 0 rpy=0 0 3.141592
- added joint r_hand_gripper_joint: type fixed, parent r_hand_force_torque, child r_hand_gripper, origin xyz=0 0.18 0 rpy=0.0 0.0 0.0
- added joint right_finger_1_joint_1: type fixed, parent right_finger_1_link_0, child right_finger_1_link_1, origin xyz=0.020 0 0 rpy=0 0 0, axis 0 0 1, limit lower=0 upper=3.1416 effort=100 velocity=100
- added joint right_finger_1_joint_2: type fixed, parent right_finger_1_link_1, child right_finger_1_link_2, origin xyz=0.050 -.028 0 rpy=0 0 -0.52, axis 0 0 1, limit lower=0 upper=3.1416 effort=100 velocity=100
- added joint right_finger_1_joint_3: type fixed, parent right_finger_1_link_2, child right_finger_1_link_3, origin xyz=0.039 0 0 rpy=0 0 0, axis 0 0 1, limit lower=0 upper=3.1416 effort=100 velocity=100
- added joint right_finger_2_joint_1: type fixed, parent right_finger_2_link_0, child right_finger_2_link_1, origin xyz=0.020 0 0 rpy=0 0 0, axis 0 0 1, limit lower=0 upper=3.1416 effort=100 velocity=100
- added joint right_finger_2_joint_2: type fixed, parent right_finger_2_link_1, child right_finger_2_link_2, origin xyz=0.050 -.028 0 rpy=0 0 -0.52, axis 0 0 1, limit lower=0 upper=3.1416 effort=100 velocity=100
- added joint right_finger_2_joint_3: type fixed, parent right_finger_2_link_2, child right_finger_2_link_3, origin xyz=0.039 0 0 rpy=0 0 0, axis 0 0 1, limit lower=0 upper=3.1416 effort=100 velocity=100
- added joint right_finger_middle_joint_1: type fixed, parent right_finger_middle_link_0, child right_finger_middle_link_1, origin xyz=0.020 0 0 rpy=0 0 0, axis 0 0 1, limit lower=0 upper=3.1416 effort=100 velocity=100
- added joint right_finger_middle_joint_2: type fixed, parent right_finger_middle_link_1, child right_finger_middle_link_2, origin xyz=0.050 -.028 0 rpy=0 0 -0.52, axis 0 0 1, limit lower=0 upper=3.1416 effort=100 velocity=100
- added joint right_finger_middle_joint_3: type fixed, parent right_finger_middle_link_2, child right_finger_middle_link_3, origin xyz=0.039 0 0 rpy=0 0 0, axis 0 0 1, limit lower=0 upper=3.1416 effort=100 velocity=100
- added joint right_palm_finger_1_joint: type fixed, parent right_palm, child right_finger_1_link_0, origin xyz=-0.0455 0.0214 0.036 rpy=0 3.1416 -1.57, axis 0 1 0, limit lower=-0.16 upper=0.25 effort=100 velocity=100
- added joint right_palm_finger_2_joint: type fixed, parent right_palm, child right_finger_2_link_0, origin xyz=-0.0455 0.0214 -0.036 rpy=0 3.1416 -1.57, axis 0 1 0, limit lower=-0.25 upper=0.16 effort=100 velocity=100
- added joint right_palm_finger_middle_joint: type fixed, parent right_palm, child right_finger_middle_link_0, origin xyz=0.0455 0.0214 0 rpy=0 0 1.57, axis 0 0 1
- added joint right_robotiq_hand_joint: type fixed, parent r_hand_force_torque, child right_palm, origin xyz=0 0.06566 0.0 rpy=0 -1.57079 0
