Commit message: Fix IRB URDF wrist direction, bugfix in rigidbodytree

File: drake/examples/IRB140/urdf/irb_140_robotiq.urdf (robot description, URDF)
Before this commit: robot IRB140, 41 links, 40 joints
Joints:
- joint joint5: axis 0 0 -1 -> 0 0 1

File: drake/examples/IRB140/urdf/irb_140_robotiq_ati.urdf (robot description, URDF)
Before this commit: robot IRB140, 42 links, 41 joints
Joints:
- joint joint5: axis 0 0 -1 -> 0 0 1
