Commit message: Fix forcetorque sensor orientation

File: drake/examples/IRB140/urdf/irb_140_robotiq_ati.urdf (robot description, URDF)
Before this commit: robot IRB140, 42 links, 41 joints
Joints:
- joint ati_joint: origin xyz=0.00953 0 0 rpy=0.0 0.0 -1.57079 -> xyz=0.00953 0 0 rpy=0.0 -2.5 -1.57079
