Commit message: Fix gelsight calib

File: drake/examples/IRB140/urdf/irb_140_robotiq_ati_invis_hand.urdf (robot description, URDF)
Before this commit: robot IRB140, 44 links, 43 joints
Links:
- link finger_middle_fourbar_linkage: geometry 
- link gelsight_box: geometry visual box size=0.033 0.033 0.031
Joints:
- joint gelsight_box_joint: origin xyz=0.105 0 0 rpy=3.1415 -1.579 0.0 -> xyz=0.09814 0 0 rpy=3.1415 -1.579 0.0
